File: batrai bor/batrai bor.kicad_sch (KiCad schematic)
At the start: 15 parts, among them J10 +, J11 +, J12 -, J13 -, J2 Molex, J3 2, J4 3, J5 4, J6 5, J8 1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

Commit message: V.4
Parts:
- removed H3, H4: Hole, MountingHole:MountingHole_3.2mm_M3_DIN965_Pad, symbol Mechanical:MountingHole
- H1, H2: footprint MountingHole:MountingHole_3.2mm_M3_DIN965_Pad -> MountingHole:MountingHole_2.2mm_M2_DIN965_Pad
