File: batrai bor/batrai bor.kicad_pcb (KiCad board)
At the start: 2 copper layers, 48.3 x 49.3 mm, 19 parts, among them J10 +, J11 +, J12 -, J13 -, J2 Molex, J3 2, J4 3, J5 4, J6 5, J8 1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

Commit message: V.4
Parts:
- removed the G*** at (70.6, 91.7)
- removed H3, H4: Hole, MountingHole:MountingHole_3.2mm_M3_DIN965_Pad
- removed kibuzzard-65E875B4: G***, kibuzzard-65E875B4
- removed kibuzzard-65E875BF: G***, kibuzzard-65E875BF
- removed kibuzzard-65E87684: G***, kibuzzard-65E87684
- added G***: LOGO, LOGO, F.Cu at (44.3, 25.1)
- added G***: LOGO, LOGO, F.Cu at (27.0, 25.1)
- H1, H2: footprint MountingHole:MountingHole_3.2mm_M3_DIN965_Pad -> MountingHole:MountingHole_2.2mm_M2_DIN965_Pad
- moved J10 78.2 mm to (56.6, 21.9)
- moved J11 78.2 mm to (52.0, 21.9)
- moved J12 78.2 mm to (19.2, 21.9)
- moved J13 78.2 mm to (14.6, 21.9)
- moved J2 78.2 mm to (29.3, 36.9)
- moved J9 77.1 mm to (54.3, 16.8)
- moved J8 75.9 mm to (16.9, 16.8)
- moved J6 73.3 mm to (47.0, 16.8)
- moved J5 72.7 mm to (39.6, 16.8)
- moved J4 72.2 mm to (32.0, 16.8)
- moved J3 71.8 mm to (24.4, 16.8)
- moved H2 71.5 mm to (35.8, 30.1)
- moved H1 57.8 mm to (35.8, 20.3)
Routing:
- net /+: track 91.5 -> 198.6 mm
- net /-: track 78.0 -> 128.1 mm
- net Net-(J2-Pin_5): track 32.0 -> 23.3 mm
- net Net-(J2-Pin_2): track 31.7 -> 23.3 mm
- net Net-(J2-Pin_3): track 27.8 -> 24.3 mm
- net Net-(J2-Pin_4): track 27.9 -> 24.9 mm
Other:
- board size 48.3 x 49.3 mm -> 47 x 33 mm
- board text added: "+"
- board text added: "-"
- board text added: "BISMILLAH"

Commit message: V.4.1
Parts:
- moved J2 13.0 mm to (38.3, 46.4)
- moved J5 12.6 mm to (49.4, 24.6)
- moved J10 12.0 mm to (65.8, 29.8)
- moved J11 12.0 mm to (61.1, 29.8)
- moved J9 12.0 mm to (63.4, 24.6)
- moved G*** 11.2 mm to (52.2, 33.0)
- moved J6 11.2 mm to (55.0, 24.6)
- moved H2 11.2 mm to (43.8, 38.0)
- moved J3 11.2 mm to (32.3, 24.6)
- moved J8 11.2 mm to (24.9, 24.6)
- moved G*** 11.2 mm to (34.9, 33.0)
- moved H1 11.2 mm to (43.8, 28.1)
- moved J12 11.1 mm to (27.0, 29.8)
- moved J13 11.1 mm to (22.4, 29.8)
- moved J4 9.85 mm to (37.9, 24.6)
Routing:
- net /-: track 128.1 -> 0.00 mm
- net /+: track 198.6 -> 193.0 mm
- net Net-(J2-Pin_2): track 23.3 -> 25.2 mm
- net Net-(J2-Pin_4): track 24.9 -> 23.2 mm
- net Net-(J2-Pin_5): track 23.3 -> 24.5 mm
Other:
- board size 47 x 33 mm -> 48 x 33 mm
